File: BoosterPack.kicad_pcb (KiCad board)
At the start: 2 copper layers, 61 parts, among them IC1 LTC4372IMS8#TRPBF, IC2 L4940D2T12-TR, IC3 MAX738ACWE+, IC4 PJ-002A, IC5 DRV103U_2K5, J1 691137710002, J2 PRT-16763, J3 691137710002, J4 53048-0810, Q1 BSC026NE2LS5ATMA1

Commit message: initial commit for layout
Parts:
- moved J1 119.2 mm to (187.3, 145.4), turned to 90 degrees
- moved J3 101.6 mm to (187.3, 126.4), turned to 90 degrees
- moved J4 92.3 mm to (188.6, 101.6), turned to 90 degrees
- moved R2 84.4 mm to (124.5, 132.7)
- moved D8 72.1 mm to (120.7, 129.5)
- moved D10 70.0 mm to (120.7, 134.6)
- moved D7 63.2 mm to (120.7, 124.5)
- moved D5 61.5 mm to (120.7, 119.4)
- moved D9 59.9 mm to (120.7, 132.1)
- moved D3 55.9 mm to (120.7, 104.1)
- moved D6 54.8 mm to (120.7, 121.9)
- moved R1 49.0 mm to (156.2, 111.1), turned to 270 degrees
- moved C1 36.4 mm to (161.3, 133.3), turned to 90 degrees
- moved Q1 32.2 mm to (150.9, 130.8), turned to 90 degrees
- moved IC1 30.9 mm to (156.2, 130.8)
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