File: SolenoidDriver.sch (KiCad schematic (older format))
At the start: 9 parts, among them IC5 DRV103U_2K5

Commit message: added connector to schematic
Parts:
- C10: footprint (none) -> Capacitor_SMD:C_0805_2012Metric_Pad1.18x1.45mm_HandSolder
- D11: footprint (none) -> Diode_SMD:D_0805_2012Metric_Pad1.15x1.40mm_HandSolder
- R3, R4, R5: footprint (none) -> Resistor_SMD:R_0805_2012Metric_Pad1.20x1.40mm_HandSolder
Changed lines of the file:
@@
 F 0 "R4" V 3993 2000 50  0000 C CNN
 F 1 "137 kiloohms" V 4084 2000 50  0000 C CNN
-F 2 "" V 4130 2000 50  0001 C CNN
+F 2 "Resistor_SMD:R_0805_2012Metric_Pad1.20x1.40mm_HandSolder" V 4130 2000 50  0001 C CNN
 F 3 "~" H 4200 2000 50  0001 C CNN
 	1    4200 2000
@@
 F 0 "C10" V 3900 2150 50  0000 C CNN
 F 1 "0.1 uF" V 4100 2200 50  0000 C CNN
-F 2 "" H 3988 2100 50  0001 C CNN
+F 2 "Capacitor_SMD:C_0805_2012Metric_Pad1.18x1.45mm_HandSolder" H 3988 2100 50  0001 C CNN
 F 3 "~" H 3950 2250 50  0001 C CNN
 	1    3950 2250
@@
 F 0 "R3" V 3900 2450 50  0000 C CNN
 F 1 "205 kiloohms" V 4050 2550 50  0000 C CNN
-F 2 "" V 3880 2600 50  0001 C CNN
+F 2 "Resistor_SMD:R_0805_2012Metric_Pad1.20x1.40mm_HandSolder" V 3880 2600 50  0001 C CNN
 F 3 "~" H 3950 2600 50  0001 C CNN
 	1    3950 2600
@@
 F 0 "D11" H 7493 2317 50  0000 C CNN
 F 1 "Low-Current LED" H 7493 2226 50  0000 C CNN
-F 2 "" H 7500 2100 50  0001 C CNN
+F 2 "Diode_SMD:D_0805_2012Metric_Pad1.15x1.40mm_HandSolder" H 7500 2100 50  0001 C CNN
 F 3 "~" H 7500 2100 50  0001 C CNN
 	1    7500 2100
@@
 F 0 "R5" H 7820 2296 50  0000 L CNN
 F 1 "5.6 kiloohms" H 7820 2205 50  0000 L CNN
-F 2 "" V 7680 2250 50  0001 C CNN
+F 2 "Resistor_SMD:R_0805_2012Metric_Pad1.20x1.40mm_HandSolder" V 7680 2250 50  0001 C CNN
 F 3 "~" H 7750 2250 50  0001 C CNN
 	1    7750 2250

Commit message: Started schematic development
Parts:
- removed R3: 205 kiloohms, Resistor_SMD:R_0805_2012Metric_Pad1.20x1.40mm_HandSolder, symbol Device:R
- added R3: MRS25000C2053FCT00, RESAD1650W60L650D250, symbol Capstone:MRS25000C2053FCT00
- C10: value 0.1 uF -> 0.1u; footprint Capacitor_SMD:C_0805_2012Metric_Pad1.18x1.45mm_HandSolder -> Capacitor_THT:C_Rect_L7.0mm_W2.5mm_P5.00mm
- C11: footprint (none) -> Capstone:CAPPRD200W52D500H1250
- R4: value 137 kiloohms -> 137k; footprint Resistor_SMD:R_0805_2012Metric_Pad1.20x1.40mm_HandSolder -> Resistor_THT:R_Axial_DIN0204_L3.6mm_D1.6mm_P7.62mm_Horizontal
- R5: value 5.6 kiloohms -> 5.6k; footprint Resistor_SMD:R_0805_2012Metric_Pad1.20x1.40mm_HandSolder -> Resistor_THT:R_Axial_DIN0204_L3.6mm_D1.6mm_P7.62mm_Horizontal
- TP22: footprint (none) -> TestPoint:TestPoint_Loop_D2.60mm_Drill1.6mm_Beaded
Connections:
- wire segments 33 -> 32
Changed lines of the file:
@@
 P 4200 2000
 F 0 "R4" V 3993 2000 50  0000 C CNN
-F 1 "137 kiloohms" V 4084 2000 50  0000 C CNN
-F 2 "Resistor_SMD:R_0805_2012Metric_Pad1.20x1.40mm_HandSolder" V 4130 2000 50  0001 C CNN
+F 1 "137k" V 4084 2000 50  0000 C CNN
+F 2 "Resistor_THT:R_Axial_DIN0204_L3.6mm_D1.6mm_P7.62mm_Horizontal" V 4130 2000 50  0001 C CNN
 F 3 "~" H 4200 2000 50  0001 C CNN
 	1    4200 2000
@@
 U 1 1 6157796B
 P 3950 2250
-F 0 "C10" V 3900 2150 50  0000 C CNN
-F 1 "0.1 uF" V 4100 2200 50  0000 C CNN
-F 2 "Capacitor_SMD:C_0805_2012Metric_Pad1.18x1.45mm_HandSolder" H 3988 2100 50  0001 C CNN
+F 0 "C10" V 3800 2150 50  0000 C CNN
+F 1 "0.1u" V 4100 2200 50  0000 C CNN
+F 2 "Capacitor_THT:C_Rect_L7.0mm_W2.5mm_P5.00mm" H 3988 2100 50  0001 C CNN
 F 3 "~" H 3950 2250 50  0001 C CNN
 	1    3950 2250
@@
 Wire Wire Line
 	4250 2600 4100 2600
-$Comp
-L Device:R R3
-U 1 1 61579346
-P 3950 2600
-F 0 "R3" V 3900 2450 50  0000 C CNN
-F 1 "205 kiloohms" V 4050 2550 50  0000 C CNN
-F 2 "Resistor_SMD:R_0805_2012Metric_Pad1.20x1.40mm_HandSolder" V 3880 2600 50  0001 C CNN
-F 3 "~" H 3950 2600 50  0001 C CNN
-	1    3950 2600
-	0    1    1    0
-$EndComp
 $Comp
 L Capstone:SD0805S020S1R0 D12
@@
 F 0 "C11" V 7100 2250 50  0000 C CNN
 F 1 "22uF" V 7000 2350 50  0000 C CNN
-F 2 "" H 7188 2200 50  0001 C CNN
+F 2 "Capstone:CAPPRD200W52D500H1250" H 7188 2200 50  0001 C CNN
 F 3 "~" H 7150 2350 50  0001 C CNN
 	1    7150 2350
@@
 P 7750 2250
 F 0 "R5" H 7820 2296 50  0000 L CNN
-F 1 "5.6 kiloohms" H 7820 2205 50  0000 L CNN
-F 2 "Resistor_SMD:R_0805_2012Metric_Pad1.20x1.40mm_HandSolder" V 7680 2250 50  0001 C CNN
+F 1 "5.6k" H 7820 2205 50  0000 L CNN
+F 2 "Resistor_THT:R_Axial_DIN0204_L3.6mm_D1.6mm_P7.62mm_Horizontal" V 7680 2250 50  0001 C CNN
 F 3 "~" H 7750 2250 50  0001 C CNN
 	1    7750 2250
@@
 L power:GND #PWR0124
 U 1 1 6164E047
-P 3550 2600
-F 0 "#PWR0124" H 3550 2350 50  0001 C CNN
-F 1 "GND" H 3555 2427 50  0000 C CNN
-F 2 "" H 3550 2600 50  0001 C CNN
-F 3 "" H 3550 2600 50  0001 C CNN
-	1    3550 2600
-	0    1    1    0
-$EndComp
-Wire Wire Line
-	3550 2600 3800 2600
+P 3400 2600
+F 0 "#PWR0124" H 3400 2350 50  0001 C CNN
+F 1 "GND" H 3405 2427 50  0000 C CNN
+F 2 "" H 3400 2600 50  0001 C CNN
+F 3 "" H 3400 2600 50  0001 C CNN
+	1    3400 2600
+	0    1    1    0
+$EndComp
 $Comp
 L power:GND #PWR0125
@@
 F 0 "TP22" H 4142 3176 50  0000 R CNN
 F 1 "GND Driver" H 4142 3267 50  0000 R CNN
-F 2 "" H 4400 3150 50  0001 C CNN
+F 2 "TestPoint:TestPoint_Loop_D2.60mm_Drill1.6mm_Beaded" H 4400 3150 50  0001 C CNN
 F 3 "~" H 4400 3150 50  0001 C CNN
 	1    4200 3150
@@
 Text Label 5250 1650 0    50   ~ 0
 Solenoid_Driver_IC
+$Comp
+L Capstone:MRS25000C2053FCT00 R3
+U 1 1 6161A6A8
+P 3400 2600
+F 0 "R3" H 3650 2700 50  0000 C CNN
+F 1 "MRS25000C2053FCT00" H 3750 2500 50  0000 C CNN
+F 2 "RESAD1650W60L650D250" H 3950 2650 50  0001 L CNN
+F 3 "http://www.vishay.com/docs/28724/mrs16m25.pdf" H 3950 2550 50  0001 L CNN
+F 4 "Vishay MRS25 Series Axial Thin Film Resistor 205k +/-1% 0.6W +/-50ppm/C" H 3950 2450 50  0001 L CNN "Description"
+F 5 "" H 3950 2350 50  0001 L CNN "Height"
+F 6 "Vishay" H 3950 2250 50  0001 L CNN "Manufacturer_Name"
+F 7 "MRS25000C2053FCT00" H 3950 2150 50  0001 L CNN "Manufacturer_Part_Number"
+F 8 "" H 3950 2050 50  0001 L CNN "Mouser Part Number"
+F 9 "" H 3950 1950 50  0001 L CNN "Mouser Price/Stock"
+F 10 "" H 3950 1850 50  0001 L CNN "Arrow Part Number"
+F 11 "" H 3950 1750 50  0001 L CNN "Arrow Price/Stock"
+	1    3400 2600
+	1    0    0    -1
+$EndComp
 $EndSCHEMATC

Commit message: initial commit for layout
Parts:
- R4, R5: footprint Resistor_THT:R_Axial_DIN0204_L3.6mm_D1.6mm_P7.62mm_Horizontal -> Capstone:RESAD1650W60L650D250
Changed lines of the file:
@@
 F 0 "R4" V 3993 2000 50  0000 C CNN
 F 1 "137k" V 4084 2000 50  0000 C CNN
-F 2 "Resistor_THT:R_Axial_DIN0204_L3.6mm_D1.6mm_P7.62mm_Horizontal" V 4130 2000 50  0001 C CNN
+F 2 "Capstone:RESAD1650W60L650D250" V 4130 2000 50  0001 C CNN
 F 3 "~" H 4200 2000 50  0001 C CNN
 	1    4200 2000
@@
 F 0 "R5" H 7820 2296 50  0000 L CNN
 F 1 "5.6k" H 7820 2205 50  0000 L CNN
-F 2 "Resistor_THT:R_Axial_DIN0204_L3.6mm_D1.6mm_P7.62mm_Horizontal" V 7680 2250 50  0001 C CNN
+F 2 "Capstone:RESAD1650W60L650D250" V 7680 2250 50  0001 C CNN
 F 3 "~" H 7750 2250 50  0001 C CNN
 	1    7750 2250
