File: SolenoidDriver.sch (KiCad schematic (older format))
At the start: 9 parts, among them IC5 DRV103U_2K5

Commit message: work on layout
Parts:
- C10: symbol Device:C -> BoosterPack-rescue:C-Device
- C11: symbol Device:CP -> BoosterPack-rescue:CP-Device
- D11: symbol Device:LED -> BoosterPack-rescue:LED-Device
- R4, R5: symbol Device:R -> BoosterPack-rescue:R-Device
- TP22: symbol Connector:TestPoint -> BoosterPack-rescue:TestPoint-Connector
Changed lines of the file:
@@
 	6950 2000 6650 2000
 $Comp
-L Device:R R4
+L BoosterPack-rescue:R-Device R4
 U 1 1 6157706B
 P 4200 2000
@@
 	4350 2000 4550 2000
 $Comp
-L Device:C C10
+L BoosterPack-rescue:C-Device C10
 U 1 1 6157796B
 P 3950 2250
@@
 Connection ~ 6950 2350
 $Comp
-L Device:CP C11
+L BoosterPack-rescue:CP-Device C11
 U 1 1 6157E351
 P 7150 2350
@@
 $EndComp
 $Comp
-L Device:LED D11
+L BoosterPack-rescue:LED-Device D11
 U 1 1 615819DE
 P 7500 2100
@@
 $EndComp
 $Comp
-L Device:R R5
+L BoosterPack-rescue:R-Device R5
 U 1 1 6158256B
 P 7750 2250
@@
 NOTE: Driver is negative logic
 $Comp
-L power:GND #PWR0124
+L BoosterPack-rescue:GND-power #PWR0124
 U 1 1 6164E047
 P 3400 2600
@@
 $EndComp
 $Comp
-L power:GND #PWR0125
+L BoosterPack-rescue:GND-power #PWR0125
 U 1 1 61651136
 P 3550 2250
@@
 $EndComp
 $Comp
-L power:GND #PWR0126
+L BoosterPack-rescue:GND-power #PWR0126
 U 1 1 616517DF
 P 3550 2000
@@
 	3550 2250 3800 2250
 $Comp
-L power:GND #PWR0127
+L BoosterPack-rescue:GND-power #PWR0127
 U 1 1 61652A81
 P 7400 2350
@@
 $EndComp
 $Comp
-L power:GND #PWR0128
+L BoosterPack-rescue:GND-power #PWR0128
 U 1 1 61654989
 P 3550 2900
@@
 	6950 1750 7050 1750
 $Comp
-L Connector:TestPoint TP?
+L BoosterPack-rescue:TestPoint-Connector TP?
 U 1 1 6185655C
 P 4200 3150
 AR Path="/61536750/6185655C" Ref="TP?"  Part="1"
 AR Path="/6153F75A/6185655C" Ref="TP22"  Part="1"
+AR Path="/6185655C" Ref="TP22"  Part="1"
 F 0 "TP22" H 4142 3176 50  0000 R CNN
 F 1 "GND Driver" H 4142 3267 50  0000 R CNN

Commit message: Finished first attempt at routing
Connections:
- wire segments 32 -> 33
Changed lines of the file:
@@
 $EndComp
 Wire Wire Line
-	3550 2900 4400 2900
+	3550 2900 4200 2900
 Wire Wire Line
 	4400 2900 4400 2300
@@
 	-1   0    0    1
 $EndComp
-Wire Wire Line
-	4200 3150 4200 2900
 Text Label 5250 1650 0    50   ~ 0
 Solenoid_Driver_IC
@@
 	1    0    0    -1
 $EndComp
+Wire Wire Line
+	4200 3150 4200 2900
+Connection ~ 4200 2900
+Wire Wire Line
+	4200 2900 4400 2900
 $EndSCHEMATC
