File: PowerPathing.sch (KiCad schematic (older format))
At the start: 23 parts, among them IC1 LTC4372IMS8#TRPBF, IC2 L4940D2T12-TR, IC3 MAX738ACWE+, Q1 BSC026NE2LS5ATMA1

Commit message: work on layout
Parts:
- C1, C3, C5, C6, C8: symbol Device:C -> BoosterPack-rescue:C-Device
- C2, C7, C9: symbol Device:CP -> BoosterPack-rescue:CP-Device
- D1: symbol Device:D -> BoosterPack-rescue:D-Device
- R1, R2: symbol Device:R -> BoosterPack-rescue:R-Device
- TP1, TP2, TP3, TP4, TP5: symbol Connector:TestPoint -> BoosterPack-rescue:TestPoint-Connector
Changed lines of the file:
@@
 $EndComp
 $Comp
-L Device:CP C9
+L BoosterPack-rescue:CP-Device C9
 U 1 1 61548B4E
 P 9400 2900
@@
 Connection ~ 7050 2450
 $Comp
-L Device:C C3
+L BoosterPack-rescue:C-Device C3
 U 1 1 6154C168
 P 4750 2800
@@
 	5650 2650 4750 2650
 $Comp
-L Device:R R2
+L BoosterPack-rescue:R-Device R2
 U 1 1 6154CCF0
 P 5400 2900
@@
 	5400 3050 5650 3050
 $Comp
-L Device:C C5
+L BoosterPack-rescue:C-Device C5
 U 1 1 6154DB48
 P 5400 3250
@@
 Connection ~ 5400 3050
 $Comp
-L Device:C C8
+L BoosterPack-rescue:C-Device C8
 U 1 1 6154E910
 P 6300 3550
@@
 Connection ~ 9400 2750
 $Comp
-L Device:C C6
+L BoosterPack-rescue:C-Device C6
 U 1 1 6156AEE8
 P 6150 4500
@@
 	5450 4500 6000 4500
 $Comp
-L Device:CP C7
+L BoosterPack-rescue:CP-Device C7
 U 1 1 6156D3FC
 P 6150 5350
@@
 Connection ~ 5450 4500
 $Comp
-L Device:CP C2
+L BoosterPack-rescue:CP-Device C2
 U 1 1 61572EC3
 P 4300 1900
@@
 $EndComp
 $Comp
-L Device:C C1
+L BoosterPack-rescue:C-Device C1
 U 1 1 615927B4
 P 3750 2850
@@
 Vin
 $Comp
-L Device:R R1
+L BoosterPack-rescue:R-Device R1
 U 1 1 615CD244
 P 1600 2050
@@
 $EndComp
 $Comp
-L Device:D D1
+L BoosterPack-rescue:D-Device D1
 U 1 1 615CDA63
 P 1300 1750
@@
 VS
 $Comp
-L Connector:TestPoint TP?
+L BoosterPack-rescue:TestPoint-Connector TP?
 U 1 1 6162E091
 P 4250 5250
 AR Path="/61536750/6162E091" Ref="TP?"  Part="1"
 AR Path="/6153BBA2/6162E091" Ref="TP2"  Part="1"
+AR Path="/6162E091" Ref="TP2"  Part="1"
 F 0 "TP2" H 4192 5276 50  0000 R CNN
 F 1 "TestPoint - 12V Reg" H 4192 5367 50  0000 R CNN
@@
 Connection ~ 5550 5050
 $Comp
-L Connector:TestPoint TP?
+L BoosterPack-rescue:TestPoint-Connector TP?
 U 1 1 6163C53C
 P 10150 2600
 AR Path="/61536750/6163C53C" Ref="TP?"  Part="1"
 AR Path="/6153BBA2/6163C53C" Ref="TP5"  Part="1"
+AR Path="/6163C53C" Ref="TP5"  Part="1"
 F 0 "TP5" H 10208 2718 50  0000 L CNN
 F 1 "TestPoint - 5V Reg" H 10208 2627 50  0000 L CNN
@@
 Connection ~ 10150 2750
 $Comp
-L Connector:TestPoint TP?
+L BoosterPack-rescue:TestPoint-Connector TP?
 U 1 1 61644C04
 P 3600 1550
 AR Path="/61536750/61644C04" Ref="TP?"  Part="1"
 AR Path="/6153BBA2/61644C04" Ref="TP1"  Part="1"
+AR Path="/61644C04" Ref="TP1"  Part="1"
 F 0 "TP1" H 3658 1668 50  0000 L CNN
 F 1 "TestPoint - Power Circuit Out" H 3658 1577 50  0000 L CNN
@@
 Connection ~ 2950 3450
 $Comp
-L power:GND #PWR0101
+L BoosterPack-rescue:GND-power #PWR0101
 U 1 1 61689C6A
 P 3750 3100
@@
 	3750 3100 3750 3000
 $Comp
-L power:GND #PWR0102
+L BoosterPack-rescue:GND-power #PWR0102
 U 1 1 6169BE0B
 P 3650 2300
@@
 	3650 2300 3550 2300
 $Comp
-L power:GND #PWR0103
+L BoosterPack-rescue:GND-power #PWR0103
 U 1 1 6169F36F
 P 3650 2500
@@
 	3650 2500 3550 2500
 $Comp
-L power:GND #PWR0104
+L BoosterPack-rescue:GND-power #PWR0104
 U 1 1 616A64FD
 P 4300 2150
@@
 	4300 2150 4300 2050
 $Comp
-L power:GND #PWR0105
+L BoosterPack-rescue:GND-power #PWR0105
 U 1 1 616ACF0A
 P 5050 2300
@@
 $EndComp
 $Comp
-L power:GND #PWR0106
+L BoosterPack-rescue:GND-power #PWR0106
 U 1 1 616B3AEC
 P 4750 3050
@@
 	4750 3050 4750 2950
 $Comp
-L power:GND #PWR0107
+L BoosterPack-rescue:GND-power #PWR0107
 U 1 1 616BA4E5
 P 5400 3500
@@
 	7100 2950 7100 3050
 $Comp
-L power:GND #PWR0108
+L BoosterPack-rescue:GND-power #PWR0108
 U 1 1 616C1223
 P 7350 3000
@@
 $EndComp
 $Comp
-L power:GND #PWR0109
+L BoosterPack-rescue:GND-power #PWR0109
 U 1 1 616C7A61
 P 9400 3150
@@
 	9850 2750 9850 3800
 $Comp
-L power:GND #PWR0110
+L BoosterPack-rescue:GND-power #PWR0110
 U 1 1 616D8001
 P 7700 3550
@@
 	7700 3550 7700 3450
 $Comp
-L power:GND #PWR0111
+L BoosterPack-rescue:GND-power #PWR0111
 U 1 1 616DE601
 P 7000 4950
@@
 	7100 3000 7350 3000
 $Comp
-L Connector:TestPoint TP?
+L BoosterPack-rescue:TestPoint-Connector TP?
 U 1 1 6184DFD4
 P 7200 3250
 AR Path="/61536750/6184DFD4" Ref="TP?"  Part="1"
 AR Path="/6153BBA2/6184DFD4" Ref="TP4"  Part="1"
+AR Path="/6184DFD4" Ref="TP4"  Part="1"
 F 0 "TP4" H 7000 3400 50  0000 L CNN
 F 1 "GND 5V Reg" H 6800 3500 50  0000 L CNN
@@
 	7200 3250 7200 3000
 $Comp
-L Connector:TestPoint TP?
+L BoosterPack-rescue:TestPoint-Connector TP?
 U 1 1 61852063
 P 7150 5150
 AR Path="/61536750/61852063" Ref="TP?"  Part="1"
 AR Path="/6153BBA2/61852063" Ref="TP3"  Part="1"
+AR Path="/61852063" Ref="TP3"  Part="1"
 F 0 "TP3" V 7104 5338 50  0000 L CNN
 F 1 "GND 12V Reg" V 7195 5338 50  0000 L CNN
