File: _autosave-BoosterPack.kicad_pcb (KiCad board)
At the start: 2 copper layers, 61 parts, among them IC1 LTC4372IMS8#TRPBF, IC2 L4940D2T12-TR, IC3 MAX738ACWE+, IC4 PJ-002A, IC5 DRV103U_2K5, J1 691137710002, J2 PRT-16763, J3 691137710002, J4 53048-0810, Q1 BSC026NE2LS5ATMA1

Commit message: work on layout
Parts:
- moved C9 65.6 mm to (199.4, 157.5), turned to 0 degrees
- moved L1 59.0 mm to (191.8, 157.5), turned to 0 degrees
- moved C3 45.8 mm to (165.1, 166.4), turned to 90 degrees
- moved IC3 18.0 mm to (177.8, 157.5)
- moved D1 14.5 mm to (124.5, 151.1)
- moved C4 2.54 mm to (167.6, 153.7), turned to 270 degrees
- turned C2 to 270 degrees
Changed lines of the file:
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@@
   )
   (module Capstone:INDPM8080X450N (layer F.Cu)
-    (at 149.86 115.93 90)
+    (at 191.77 157.48)
     (descr SRN8040TA-101M)
     (tags Inductor)
     (attr smd)
-    (fp_text reference L1 (at 0 0 90) (layer F.SilkS)
-      (effects (font (size 1.27 1.27) (thickness 0.254)))
-    )
-    (fp_text value SRN8040TA-101M (at 0 0 90) (layer F.SilkS) hide
+    (fp_text reference L1 (at 0 0) (layer F.SilkS)
+      (effects (font (size 1.27 1.27) (thickness 0.254)))
+    )
+    (fp_text value SRN8040TA-101M (at 0 0) (layer F.SilkS) hide
       (effects (font (size 1.27 1.27) (thickness 0.254)))
     )
@@
     (fp_line (start 4 -4) (end -4 -4) (layer F.SilkS) (width 0.2))
     (fp_line (start -4 4) (end 4 4) (layer F.SilkS) (width 0.2))
-    (fp_text user %R (at 0 0 90) (layer F.Fab)
-      (effects (font (size 1.27 1.27) (thickness 0.254)))
-    )
-    (pad 2 smd rect (at 2.9 0 90) (size 3.45 6.5) (layers F.Cu F.Paste F.Mask)
+    (fp_text user %R (at 0 0) (layer F.Fab)
+      (effects (font (size 1.27 1.27) (thickness 0.254)))
+    )
+    (pad 2 smd rect (at 2.9 0) (size 3.45 6.5) (layers F.Cu F.Paste F.Mask)
       (net 8 /Connectors/5V_Reg))
-    (pad 1 smd rect (at -2.9 0 90) (size 3.45 6.5) (layers F.Cu F.Paste F.Mask)
+    (pad 1 smd rect (at -2.9 0) (size 3.45 6.5) (layers F.Cu F.Paste F.Mask)
       (net 11 "Net-(D2-Pad1)"))
     (model "C:\\Users\\chros\\Documents\\ECE Capstone\\Hardware\\Libraries\\SamacSys_Parts.3dshapes\\SRN8040TA-101M.stp"
@@
   )
   (module Capstone:SOIC127P1032X265-16N (layer F.Cu)
-    (at 165.1 170.18)
+    (at 177.8 157.48)
     (descr "16 Wide SO")
     (tags "Integrated Circuit")
@@
   )
   (module Diode_SMD:D_0805_2012Metric_Pad1.15x1.40mm_HandSolder (layer F.Cu)
-    (at 120.65 137.16)
+    (at 124.46 151.13)
     (descr "Diode SMD 0805 (2012 Metric), square (rectangular) end terminal, IPC_7351 nominal, (Body size source: https://docs.google.com/spreadsheets/d/1BsfQQcO9C6DZCsRaXUlFlo91Tg2WpOkGARC1WS5S8t0/edit?usp=sharing), generated with kicad-footprint-generator")
     (tags "diode handsolder")
@@
   )
   (module Capstone:CAPPRD200W52D500H1250 (layer F.Cu)
-    (at 141.605 126.365 180)
+    (at 199.39 157.48)
     (descr 860020672005)
     (tags Capacitor)
@@
       (effects (font (size 1.27 1.27) (thickness 0.254)))
     )
-    (pad 2 thru_hole circle (at 2 0 180) (size 1.1 1.1) (drill 0.7) (layers *.Cu *.Mask)
-      (net 2 GND))
-    (pad 1 thru_hole rect (at 0 0 180) (size 1.1 1.1) (drill 0.7) (layers *.Cu *.Mask)
+    (pad 2 thru_hole circle (at 2 0) (size 1.1 1.1) (drill 0.7) (layers *.Cu *.Mask)
+      (net 2 GND))
+    (pad 1 thru_hole rect (at 0 0) (size 1.1 1.1) (drill 0.7) (layers *.Cu *.Mask)
       (net 8 /Connectors/5V_Reg))
     (model "C:\\Users\\chros\\Documents\\ECE Capstone\\Hardware\\Libraries\\SamacSys_Parts.3dshapes\\860020672005.stp"
@@
   )
   (module Capstone:CAPPRD200W52D500H1250 (layer F.Cu)
-    (at 170.18 153.67 90)
+    (at 167.64 153.67 270)
     (descr 860020672005)
     (tags Capacitor)
@@
       (effects (font (size 1.27 1.27) (thickness 0.254)))
     )
-    (pad 2 thru_hole circle (at 2 0 90) (size 1.1 1.1) (drill 0.7) (layers *.Cu *.Mask)
-      (net 2 GND))
-    (pad 1 thru_hole rect (at 0 0 90) (size 1.1 1.1) (drill 0.7) (layers *.Cu *.Mask)
+    (pad 2 thru_hole circle (at 2 0 270) (size 1.1 1.1) (drill 0.7) (layers *.Cu *.Mask)
+      (net 2 GND))
+    (pad 1 thru_hole rect (at 0 0 270) (size 1.1 1.1) (drill 0.7) (layers *.Cu *.Mask)
       (net 3 "Net-(C2-Pad1)"))
     (model "C:\\Users\\chros\\Documents\\ECE Capstone\\Hardware\\Libraries\\SamacSys_Parts.3dshapes\\860020672005.stp"
@@
   )
   (module Capacitor_THT:C_Rect_L7.0mm_W2.5mm_P5.00mm (layer F.Cu)
-    (at 127 140.97 270)
+    (at 165.1 166.37 90)
     (descr "C, Rect series, Radial, pin pitch=5.00mm, , length*width=7*2.5mm^2, Capacitor")
     (tags "C Rect series Radial pin pitch 5.00mm  length 7mm width 2.5mm Capacitor")
@@
       (effects (font (size 1 1) (thickness 0.15)))
     )
-    (pad 2 thru_hole circle (at 5 0 270) (size 1.6 1.6) (drill 0.8) (layers *.Cu *.Mask)
-      (net 2 GND))
-    (pad 1 thru_hole circle (at 0 0 270) (size 1.6 1.6) (drill 0.8) (layers *.Cu *.Mask)
+    (pad 2 thru_hole circle (at 5 0 90) (size 1.6 1.6) (drill 0.8) (layers *.Cu *.Mask)
+      (net 2 GND))
+    (pad 1 thru_hole circle (at 0 0 90) (size 1.6 1.6) (drill 0.8) (layers *.Cu *.Mask)
       (net 4 "Net-(C3-Pad1)"))
     (model ${KISYS3DMOD}/Capacitor_THT.3dshapes/C_Rect_L7.0mm_W2.5mm_P5.00mm.wrl
@@
   )
   (module Capstone:CAPPRD200W52D500H1250 (layer F.Cu)
-    (at 161.29 153.67 90)
+    (at 161.29 153.67 270)
     (descr 860020672005)
     (tags Capacitor)
@@
       (effects (font (size 1.27 1.27) (thickness 0.254)))
     )
-    (pad 2 thru_hole circle (at 2 0 90) (size 1.1 1.1) (drill 0.7) (layers *.Cu *.Mask)
-      (net 2 GND))
-    (pad 1 thru_hole rect (at 0 0 90) (size 1.1 1.1) (drill 0.7) (layers *.Cu *.Mask)
+    (pad 2 thru_hole circle (at 2 0 270) (size 1.1 1.1) (drill 0.7) (layers *.Cu *.Mask)
+      (net 2 GND))
+    (pad 1 thru_hole rect (at 0 0 270) (size 1.1 1.1) (drill 0.7) (layers *.Cu *.Mask)
       (net 3 "Net-(C2-Pad1)"))
     (model "C:\\Users\\chros\\Documents\\ECE Capstone\\Hardware\\Libraries\\SamacSys_Parts.3dshapes\\860020672005.stp"
