File: Connectors.sch (KiCad schematic (older format))
At the start: 2 parts

Commit message: Schematic Updates
Parts:
- removed IC?: PJ-002A, PJ002A, symbol Capstone:PJ-002A
- added IC?: PJ-002A, PJ002A, symbol Capstone:PJ-002A
- added J? (x2): 691137710002, SHDR2W70P0X500_1X2_1000X750X1160P, symbol Capstone:691137710002
- added TP?: TestPoint - Power Suppply, symbol Connector:TestPoint
- added TP?: TestPoint - Rechargeable Batteries, symbol Connector:TestPoint
- added TP?: TestPoint - Electric Strike, symbol Connector:TestPoint
Connections:
- net labels added: Electric_Strike, Power_Supply, Rechargeable_Batteries
- wire segments 9 -> 22
Changed lines of the file:
@@
-	1    0    0    -1
-$EndComp
-$Comp
-L Capstone:PJ-002A IC?
-U 1 1 6153AA7B
-P 5000 4600
-F 0 "IC?" H 5400 4865 50  0000 C CNN
-F 1 "PJ-002A" H 5400 4774 50  0000 C CNN
-F 2 "PJ002A" H 5650 4700 50  0001 L CNN
-F 3 "https://www.cui.com/product/resource/digikeypdf/pj-002a.pdf" H 5650 4600 50  0001 L CNN
-F 4 "CONN PWR JACK 2X5.5MM SOLDER" H 5650 4500 50  0001 L CNN "Description"
-F 5 "11" H 5650 4400 50  0001 L CNN "Height"
-F 6 "CUI Inc." H 5650 4300 50  0001 L CNN "Manufacturer_Name"
-F 7 "PJ-002A" H 5650 4200 50  0001 L CNN "Manufacturer_Part_Number"
-F 8 "490-PJ-002A" H 5650 4100 50  0001 L CNN "Mouser Part Number"
-F 9 "https://www.mouser.co.uk/ProductDetail/CUI-Devices/PJ-002A?qs=WyjlAZoYn51CKfAix9Mngw%3D%3D" H 5650 4000 50  0001 L CNN "Mouser Price/Stock"
-F 10 "PJ-002A" H 5650 3900 50  0001 L CNN "Arrow Part Number"
-F 11 "https://www.arrow.com/en/products/pj-002a/cui-devices" H 5650 3800 50  0001 L CNN "Arrow Price/Stock"
-	1    5000 4600
 	1    0    0    -1
 $EndComp
@@
 Text Label 6150 3300 2    50   ~ 0
 GND
+$Comp
+L Capstone:691137710002 J?
+U 1 1 615C9DB6
+P 2450 2650
+F 0 "J?" H 3078 2646 50  0000 L CNN
+F 1 "691137710002" H 3078 2555 50  0000 L CNN
+F 2 "SHDR2W70P0X500_1X2_1000X750X1160P" H 3100 2750 50  0001 L CNN
+F 3 "https://katalog.we-online.com/em/datasheet/691137710002.pdf" H 3100 2650 50  0001 L CNN
+F 4 "Wurth Elektronik WR-TBL Series 5mm Pitch, 2 Way, PCB Terminal Block, Through Hole" H 3100 2550 50  0001 L CNN "Description"
+F 5 "11.6" H 3100 2450 50  0001 L CNN "Height"
+F 6 "Wurth Elektronik" H 3100 2350 50  0001 L CNN "Manufacturer_Name"
+F 7 "691137710002" H 3100 2250 50  0001 L CNN "Manufacturer_Part_Number"
+F 8 "710-691137710002" H 3100 2150 50  0001 L CNN "Mouser Part Number"
+F 9 "https://www.mouser.co.uk/ProductDetail/Wurth-Elektronik/691137710002?qs=lBTPRtX1sU9LnHBbviNKGA%3D%3D" H 3100 2050 50  0001 L CNN "Mouser Price/Stock"
+	1    2450 2650
+	1    0    0    -1
+$EndComp
+$Comp
+L Capstone:691137710002 J?
+U 1 1 615CAB9C
+P 7800 2250
+F 0 "J?" H 8428 2246 50  0000 L CNN
+F 1 "691137710002" H 8428 2155 50  0000 L CNN
+F 2 "SHDR2W70P0X500_1X2_1000X750X1160P" H 8450 2350 50  0001 L CNN
+F 3 "https://katalog.we-online.com/em/datasheet/691137710002.pdf" H 8450 2250 50  0001 L CNN
+F 4 "Wurth Elektronik WR-TBL Series 5mm Pitch, 2 Way, PCB Terminal Block, Through Hole" H 8450 2150 50  0001 L CNN "Description"
+F 5 "11.6" H 8450 2050 50  0001 L CNN "Height"
+F 6 "Wurth Elektronik" H 8450 1950 50  0001 L CNN "Manufacturer_Name"
+F 7 "691137710002" H 8450 1850 50  0001 L CNN "Manufacturer_Part_Number"
+F 8 "710-691137710002" H 8450 1750 50  0001 L CNN "Mouser Part Number"
+F 9 "https://www.mouser.co.uk/ProductDetail/Wurth-Elektronik/691137710002?qs=lBTPRtX1sU9LnHBbviNKGA%3D%3D" H 8450 1650 50  0001 L CNN "Mouser Price/Stock"
+	1    7800 2250
+	1    0    0    -1
+$EndComp
+Wire Wire Line
+	2100 2750 2450 2750
+Text Label 2100 2750 0    50   ~ 0
+GND
+Wire Wire Line
+	7450 2350 7800 2350
+Text Label 7450 2350 0    50   ~ 0
+GND
+$Comp
+L Capstone:PJ-002A IC?
+U 1 1 6160CEBD
+P 2050 1800
+F 0 "IC?" H 2450 2065 50  0000 C CNN
+F 1 "PJ-002A" H 2450 1974 50  0000 C CNN
+F 2 "PJ002A" H 2700 1900 50  0001 L CNN
+F 3 "https://www.cui.com/product/resource/digikeypdf/pj-002a.pdf" H 2700 1800 50  0001 L CNN
+F 4 "CONN PWR JACK 2X5.5MM SOLDER" H 2700 1700 50  0001 L CNN "Description"
+F 5 "11" H 2700 1600 50  0001 L CNN "Height"
+F 6 "CUI Inc." H 2700 1500 50  0001 L CNN "Manufacturer_Name"
+F 7 "PJ-002A" H 2700 1400 50  0001 L CNN "Manufacturer_Part_Number"
+F 8 "490-PJ-002A" H 2700 1300 50  0001 L CNN "Mouser Part Number"
+F 9 "https://www.mouser.co.uk/ProductDetail/CUI-Devices/PJ-002A?qs=WyjlAZoYn51CKfAix9Mngw%3D%3D" H 2700 1200 50  0001 L CNN "Mouser Price/Stock"
+F 10 "PJ-002A" H 2700 1100 50  0001 L CNN "Arrow Part Number"
+F 11 "https://www.arrow.com/en/products/pj-002a/cui-devices" H 2700 1000 50  0001 L CNN "Arrow Price/Stock"
+	1    2050 1800
+	1    0    0    -1
+$EndComp
+Wire Wire Line
+	1700 1800 2050 1800
+Text Label 1700 1800 0    50   ~ 0
+GND
+Wire Wire Line
+	3200 1800 2850 1800
+Text Label 3200 1800 2    50   ~ 0
+GND
+Text HLabel 3200 1900 2    50   Output ~ 0
+Power_Supply
+Text HLabel 1950 2650 0    50   Output ~ 0
+Rechargeable_Batteries
+Text HLabel 7350 2250 0    50   Output ~ 0
+Electric_Strike
+$Comp
+L Connector:TestPoint TP?
+U 1 1 61624CC1
+P 3050 2000
+F 0 "TP?" H 2992 2026 50  0000 R CNN
+F 1 "TestPoint - Power Suppply" H 2992 2117 50  0000 R CNN
+F 2 "" H 3250 2000 50  0001 C CNN
+F 3 "~" H 3250 2000 50  0001 C CNN
+	1    3050 2000
+	-1   0    0    1
+$EndComp
+$Comp
+L Connector:TestPoint TP?
+U 1 1 61627D05
+P 2200 2450
+F 0 "TP?" H 2258 2568 50  0000 L CNN
+F 1 "TestPoint - Rechargeable Batteries" H 2258 2477 50  0000 L CNN
+F 2 "" H 2400 2450 50  0001 C CNN
+F 3 "~" H 2400 2450 50  0001 C CNN
+	1    2200 2450
+	1    0    0    -1
+$EndComp
+Wire Wire Line
+	1950 2650 2200 2650
+Wire Wire Line
+	2200 2650 2200 2450
+Wire Wire Line
+	2450 2650 2200 2650
+Connection ~ 2200 2650
+$Comp
+L Connector:TestPoint TP?
+U 1 1 6162AC3A
+P 7550 2100
+F 0 "TP?" H 7608 2218 50  0000 L CNN
+F 1 "TestPoint - Electric Strike" H 7608 2127 50  0000 L CNN
+F 2 "" H 7750 2100 50  0001 C CNN
+F 3 "~" H 7750 2100 50  0001 C CNN
+	1    7550 2100
+	1    0    0    -1
+$EndComp
+Wire Wire Line
+	7350 2250 7550 2250
+Wire Wire Line
+	7550 2250 7550 2100
+Wire Wire Line
+	7800 2250 7550 2250
+Connection ~ 7550 2250
+Wire Wire Line
+	2850 1900 3050 1900
+Wire Wire Line
+	3050 2000 3050 1900
+Connection ~ 3050 1900
+Wire Wire Line
+	3050 1900 3200 1900
 $EndSCHEMATC

Commit message: Schematic Updates, still need component values for driver circuit and keypad connector EDA
Parts:
- added D? (x8): ESDALC6V1-1U2, ESDALC6V11U2, symbol Capstone:ESDALC6V1-1U2
- added TP?: Keypad 8, symbol Connector:TestPoint
- added TP?: Keypad 7, symbol Connector:TestPoint
- added TP?: Keypad 6, symbol Connector:TestPoint
- added TP?: Keypad 5, symbol Connector:TestPoint
- added TP?: Keypad 4, symbol Connector:TestPoint
- added TP?: Keypad 3, symbol Connector:TestPoint
- added TP?: Keypad 2, symbol Connector:TestPoint
- added TP?: Keypad 1, symbol Connector:TestPoint
- added TP?: TestPoint - Electric Strike Control, symbol Connector:TestPoint
- added TP?: TestPoint - GND Rechargeable Batteries, symbol Connector:TestPoint
- added TP?: TestPoint - GND VCC, symbol Connector:TestPoint
- added TP? (x2): GND Keypad, symbol Connector:TestPoint
- J? (x2): symbol Capstone:691137710002 -> BoosterPack-rescue:691137710002-Capstone-BoosterPack-rescue
- TP?: value TestPoint - Electric Strike -> TestPoint - Electric Strike VS
Connections:
- net labels added: 5V_Reg, Control, Keypad_Connector, Solenoid_Driver_Input, VCC, VS
- net labels removed: Electric_Strike, Power_Supply
- wire segments 22 -> 113
Other:
- moved on the sheet: IC?, J?, TP?

Commit message: Added Generic Keypad Connector, don't know if we can use it or not
Parts:
- added J4: Keypad Connector 01x08_Female, symbol Connector:Conn_01x08_Female
- gave numbers to parts that had none: 28
Connections:
- net labels removed: Keypad_Connector

Commit message: Added labels for ease of reading and reorganized a sheet, still have a Generic Keypad Connector, don't know if we can use it or not
Parts:
- TP9: value TestPoint - Power Suppply -> TestPoint - Power Supply
Connections:
- net labels added: Electric_Strike_Connector, Keypad_Connector, Power_Supply_Barrel_Jack, Raspberry_Pi_Connector, Rechageable_Batteries_Connector
Other:
- moved on the sheet: IC4, J1, J3, TP10, TP11, TP6, TP7, TP8, TP9

Commit message: added connector to schematic
Parts:
- removed J4: Keypad Connector 01x08_Female, symbol Connector:Conn_01x08_Female
- added J4: 53048-0810, 530480810, symbol Capstone:53048-0810
- TP12: value Keypad 8 -> Keypad 1
- TP13: value Keypad 7 -> Keypad 2
- TP15: value Keypad 6 -> Keypad 3
- TP16: value Keypad 5 -> Keypad 4
- TP17: value Keypad 4 -> Keypad 5
- TP18: value Keypad 3 -> Keypad 6
- TP20: value Keypad 2 -> Keypad 7
- TP21: value Keypad 1 -> Keypad 8
Changed lines of the file:
@@
 P 6600 3450
 F 0 "TP12" V 6795 3522 50  0000 C CNN
-F 1 "Keypad 8" V 6700 3600 50  0000 C CNN
+F 1 "Keypad 1" V 6700 3600 50  0000 C CNN
 F 2 "" H 6800 3450 50  0001 C CNN
 F 3 "~" H 6800 3450 50  0001 C CNN
@@
 P 7200 3450
 F 0 "TP13" V 7395 3522 50  0000 C CNN
-F 1 "Keypad 7" V 7300 3600 50  0000 C CNN
+F 1 "Keypad 2" V 7300 3600 50  0000 C CNN
 F 2 "" H 7400 3450 50  0001 C CNN
 F 3 "~" H 7400 3450 50  0001 C CNN
@@
 P 7750 3450
 F 0 "TP15" V 7945 3522 50  0000 C CNN
-F 1 "Keypad 6" V 7850 3600 50  0000 C CNN
+F 1 "Keypad 3" V 7850 3600 50  0000 C CNN
 F 2 "" H 7950 3450 50  0001 C CNN
 F 3 "~" H 7950 3450 50  0001 C CNN
@@
 P 8350 3450
 F 0 "TP16" V 8545 3522 50  0000 C CNN
-F 1 "Keypad 5" V 8450 3600 50  0000 C CNN
+F 1 "Keypad 4" V 8450 3600 50  0000 C CNN
 F 2 "" H 8550 3450 50  0001 C CNN
 F 3 "~" H 8550 3450 50  0001 C CNN
@@
 P 8850 3450
 F 0 "TP17" V 9045 3522 50  0000 C CNN
-F 1 "Keypad 4" V 8950 3600 50  0000 C CNN
+F 1 "Keypad 5" V 8950 3600 50  0000 C CNN
 F 2 "" H 9050 3450 50  0001 C CNN
 F 3 "~" H 9050 3450 50  0001 C CNN
@@
 P 9450 3450
 F 0 "TP18" V 9645 3522 50  0000 C CNN
-F 1 "Keypad 3" V 9550 3600 50  0000 C CNN
+F 1 "Keypad 6" V 9550 3600 50  0000 C CNN
 F 2 "" H 9650 3450 50  0001 C CNN
 F 3 "~" H 9650 3450 50  0001 C CNN
@@
 P 10050 3450
 F 0 "TP20" V 10245 3522 50  0000 C CNN
-F 1 "Keypad 2" V 10150 3600 50  0000 C CNN
+F 1 "Keypad 7" V 10150 3600 50  0000 C CNN
 F 2 "" H 10250 3450 50  0001 C CNN
 F 3 "~" H 10250 3450 50  0001 C CNN
@@
 P 10650 3450
 F 0 "TP21" V 10845 3522 50  0000 C CNN
-F 1 "Keypad 1" V 10750 3600 50  0000 C CNN
+F 1 "Keypad 8" V 10750 3600 50  0000 C CNN
 F 2 "" H 10850 3450 50  0001 C CNN
 F 3 "~" H 10850 3450 50  0001 C CNN
@@
 Wire Wire Line
 	4850 3950 6650 3950
-$Comp
-L Connector:Conn_01x08_Female J4
-U 1 1 615E2A19
-P 4650 4350
-F 0 "J4" H 4542 3725 50  0000 C CNN
-F 1 "Keypad Connector 01x08_Female" H 4542 3816 50  0000 C CNN
-F 2 "" H 4650 4350 50  0001 C CNN
-F 3 "~" H 4650 4350 50  0001 C CNN
-	1    4650 4350
-	-1   0    0    1
-$EndComp
 Wire Wire Line
 	3450 5150 10700 5150
@@
 Text Label 5050 3650 2    50   ~ 0
 Keypad_Connector
+$Comp
+L Capstone:53048-0810 J4
+U 1 1 615E5D56
+P 4850 4650
+F 0 "J4" H 5142 3685 50  0000 C CNN
+F 1 "53048-0810" H 5142 3776 50  0000 C CNN
+F 2 "530480810" H 5500 4750 50  0001 L CNN
+F 3 "https://www.molex.com/pdm_docs/sd/530480810_sd.pdf" H 5500 4650 50  0001 L CNN
+F 4 "8CKT R/A WAFER ASSY ROHS COMPLIANT: YES" H 5500 4550 50  0001 L CNN "Description"
+F 5 "3.7" H 5500 4450 50  0001 L CNN "Height"
+F 6 "Molex" H 5500 4350 50  0001 L CNN "Manufacturer_Name"
+F 7 "53048-0810" H 5500 4250 50  0001 L CNN "Manufacturer_Part_Number"
+F 8 "" H 5500 4150 50  0001 L CNN "Mouser Part Number"
+F 9 "" H 5500 4050 50  0001 L CNN "Mouser Price/Stock"
+F 10 "" H 5500 3950 50  0001 L CNN "Arrow Part Number"
+F 11 "" H 5500 3850 50  0001 L CNN "Arrow Price/Stock"
+	1    4850 4650
+	-1   0    0    1
+$EndComp
 $EndSCHEMATC

Commit message: Started schematic development
Parts:
- TP10, TP11, TP12, TP13, TP14, TP15, TP16, TP17, TP18, TP19, TP20, TP21, TP6, TP7, TP8, TP9: footprint (none) -> TestPoint:TestPoint_Loop_D2.60mm_Drill1.6mm_Beaded
Changed lines of the file:
@@
 F 0 "TP9" H 2092 1676 50  0000 R CNN
 F 1 "TestPoint - Power Supply" H 2650 1900 50  0000 R CNN
-F 2 "" H 2350 1650 50  0001 C CNN
+F 2 "TestPoint:TestPoint_Loop_D2.60mm_Drill1.6mm_Beaded" H 2350 1650 50  0001 C CNN
 F 3 "~" H 2350 1650 50  0001 C CNN
 	1    2150 1650
@@
 F 0 "TP6" H 1858 2768 50  0000 L CNN
 F 1 "TestPoint - Rechargeable Batteries" H 1150 2900 50  0000 L CNN
-F 2 "" H 2000 2650 50  0001 C CNN
+F 2 "TestPoint:TestPoint_Loop_D2.60mm_Drill1.6mm_Beaded" H 2000 2650 50  0001 C CNN
 F 3 "~" H 2000 2650 50  0001 C CNN
 	1    1800 2650
@@
 F 0 "TP10" H 1708 4418 50  0000 L CNN
 F 1 "TestPoint - Electric Strike VS" H 1100 4550 50  0000 L CNN
-F 2 "" H 1850 4300 50  0001 C CNN
+F 2 "TestPoint:TestPoint_Loop_D2.60mm_Drill1.6mm_Beaded" H 1850 4300 50  0001 C CNN
 F 3 "~" H 1850 4300 50  0001 C CNN
 	1    1650 4300
@@
 F 0 "TP12" V 6795 3522 50  0000 C CNN
 F 1 "Keypad 1" V 6700 3600 50  0000 C CNN
-F 2 "" H 6800 3450 50  0001 C CNN
+F 2 "TestPoint:TestPoint_Loop_D2.60mm_Drill1.6mm_Beaded" H 6800 3450 50  0001 C CNN
 F 3 "~" H 6800 3450 50  0001 C CNN
 	1    6600 3450
@@
 F 0 "TP13" V 7395 3522 50  0000 C CNN
 F 1 "Keypad 2" V 7300 3600 50  0000 C CNN
-F 2 "" H 7400 3450 50  0001 C CNN
+F 2 "TestPoint:TestPoint_Loop_D2.60mm_Drill1.6mm_Beaded" H 7400 3450 50  0001 C CNN
 F 3 "~" H 7400 3450 50  0001 C CNN
 	1    7200 3450
@@
 F 0 "TP15" V 7945 3522 50  0000 C CNN
 F 1 "Keypad 3" V 7850 3600 50  0000 C CNN
-F 2 "" H 7950 3450 50  0001 C CNN
+F 2 "TestPoint:TestPoint_Loop_D2.60mm_Drill1.6mm_Beaded" H 7950 3450 50  0001 C CNN
 F 3 "~" H 7950 3450 50  0001 C CNN
 	1    7750 3450
@@
 F 0 "TP16" V 8545 3522 50  0000 C CNN
 F 1 "Keypad 4" V 8450 3600 50  0000 C CNN
-F 2 "" H 8550 3450 50  0001 C CNN
+F 2 "TestPoint:TestPoint_Loop_D2.60mm_Drill1.6mm_Beaded" H 8550 3450 50  0001 C CNN
 F 3 "~" H 8550 3450 50  0001 C CNN
 	1    8350 3450
@@
 F 0 "TP17" V 9045 3522 50  0000 C CNN
 F 1 "Keypad 5" V 8950 3600 50  0000 C CNN
-F 2 "" H 9050 3450 50  0001 C CNN
+F 2 "TestPoint:TestPoint_Loop_D2.60mm_Drill1.6mm_Beaded" H 9050 3450 50  0001 C CNN
 F 3 "~" H 9050 3450 50  0001 C CNN
 	1    8850 3450
@@
 F 0 "TP18" V 9645 3522 50  0000 C CNN
 F 1 "Keypad 6" V 9550 3600 50  0000 C CNN
-F 2 "" H 9650 3450 50  0001 C CNN
+F 2 "TestPoint:TestPoint_Loop_D2.60mm_Drill1.6mm_Beaded" H 9650 3450 50  0001 C CNN
 F 3 "~" H 9650 3450 50  0001 C CNN
 	1    9450 3450
@@
 F 0 "TP20" V 10245 3522 50  0000 C CNN
 F 1 "Keypad 7" V 10150 3600 50  0000 C CNN
-F 2 "" H 10250 3450 50  0001 C CNN
+F 2 "TestPoint:TestPoint_Loop_D2.60mm_Drill1.6mm_Beaded" H 10250 3450 50  0001 C CNN
 F 3 "~" H 10250 3450 50  0001 C CNN
 	1    10050 3450
@@
 F 0 "TP21" V 10845 3522 50  0000 C CNN
 F 1 "Keypad 8" V 10750 3600 50  0000 C CNN
-F 2 "" H 10850 3450 50  0001 C CNN
+F 2 "TestPoint:TestPoint_Loop_D2.60mm_Drill1.6mm_Beaded" H 10850 3450 50  0001 C CNN
 F 3 "~" H 10850 3450 50  0001 C CNN
 	1    10650 3450
@@
 F 0 "TP11" H 1708 4868 50  0000 L CNN
 F 1 "TestPoint - Electric Strike Control" H 1000 5000 50  0000 L CNN
-F 2 "" H 1850 4750 50  0001 C CNN
+F 2 "TestPoint:TestPoint_Loop_D2.60mm_Drill1.6mm_Beaded" H 1850 4750 50  0001 C CNN
 F 3 "~" H 1850 4750 50  0001 C CNN
 	1    1650 4750
@@
 F 0 "TP7" H 1858 3218 50  0000 L CNN
 F 1 "TestPoint - GND Rechargeable Batteries" H 1000 3350 50  0000 L CNN
-F 2 "" H 2000 3100 50  0001 C CNN
+F 2 "TestPoint:TestPoint_Loop_D2.60mm_Drill1.6mm_Beaded" H 2000 3100 50  0001 C CNN
 F 3 "~" H 2000 3100 50  0001 C CNN
 	1    1800 3100
@@
 F 0 "TP8" H 2208 1468 50  0000 L CNN
 F 1 "TestPoint - GND VCC" H 1750 1600 50  0000 L CNN
-F 2 "" H 2350 1350 50  0001 C CNN
+F 2 "TestPoint:TestPoint_Loop_D2.60mm_Drill1.6mm_Beaded" H 2350 1350 50  0001 C CNN
 F 3 "~" H 2350 1350 50  0001 C CNN
 	1    2150 1350
@@
 F 0 "TP14" H 7608 2018 50  0000 L CNN
 F 1 "GND Keypad" H 7608 1927 50  0000 L CNN
-F 2 "" H 7750 1900 50  0001 C CNN
+F 2 "TestPoint:TestPoint_Loop_D2.60mm_Drill1.6mm_Beaded" H 7750 1900 50  0001 C CNN
 F 3 "~" H 7750 1900 50  0001 C CNN
 	1    7550 1900
@@
 F 0 "TP19" H 9808 2018 50  0000 L CNN
 F 1 "GND Keypad" H 9808 1927 50  0000 L CNN
-F 2 "" H 9950 1900 50  0001 C CNN
+F 2 "TestPoint:TestPoint_Loop_D2.60mm_Drill1.6mm_Beaded" H 9950 1900 50  0001 C CNN
 F 3 "~" H 9950 1900 50  0001 C CNN
 	1    9750 1900

Commit message: work on layout
Parts:
- TP10, TP11, TP12, TP13, TP14, TP15, TP16, TP17, TP18, TP19, TP20, TP21, TP6, TP7, TP8, TP9: symbol Connector:TestPoint -> BoosterPack-rescue:TestPoint-Connector
Changed lines of the file:
@@
 VS
 $Comp
-L Connector:TestPoint TP9
+L BoosterPack-rescue:TestPoint-Connector TP9
 U 1 1 61624CC1
 P 2150 1650
+AR Path="/61624CC1" Ref="TP9"  Part="1"
+AR Path="/61536750/61624CC1" Ref="TP9"  Part="1"
 F 0 "TP9" H 2092 1676 50  0000 R CNN
 F 1 "TestPoint - Power Supply" H 2650 1900 50  0000 R CNN
@@
 $EndComp
 $Comp
-L Connector:TestPoint TP6
+L BoosterPack-rescue:TestPoint-Connector TP6
 U 1 1 61627D05
 P 1800 2650
+AR Path="/61627D05" Ref="TP6"  Part="1"
+AR Path="/61536750/61627D05" Ref="TP6"  Part="1"
 F 0 "TP6" H 1858 2768 50  0000 L CNN
 F 1 "TestPoint - Rechargeable Batteries" H 1150 2900 50  0000 L CNN
@@
 Connection ~ 1800 2850
 $Comp
-L Connector:TestPoint TP10
+L BoosterPack-rescue:TestPoint-Connector TP10
 U 1 1 6162AC3A
 P 1650 4300
+AR Path="/6162AC3A" Ref="TP10"  Part="1"
+AR Path="/61536750/6162AC3A" Ref="TP10"  Part="1"
 F 0 "TP10" H 1708 4418 50  0000 L CNN
 F 1 "TestPoint - Electric Strike VS" H 1100 4550 50  0000 L CNN
@@
 	5400 1200 5600 1200
 $Comp
-L power:GND #PWR0112
+L BoosterPack-rescue:GND-power #PWR0112
 U 1 1 61736CD0
 P 4350 3100
@@
 $EndComp
 $Comp
-L power:GND #PWR0113
+L BoosterPack-rescue:GND-power #PWR0113
 U 1 1 61737540
 P 4300 2400
@@
 $EndComp
 $Comp
-L power:GND #PWR0114
+L BoosterPack-rescue:GND-power #PWR0114
 U 1 1 61737FC4
 P 4300 1600
@@
 	5850 1400 5400 1400
 $Comp
-L power:GND #PWR0115
+L BoosterPack-rescue:GND-power #PWR0115
 U 1 1 61735922
 P 5850 2800
@@
 $EndComp
 $Comp
-L power:GND #PWR0116
+L BoosterPack-rescue:GND-power #PWR0116
 U 1 1 61734F70
 P 5850 2600
@@
 $EndComp
 $Comp
-L power:GND #PWR0117
+L BoosterPack-rescue:GND-power #PWR0117
 U 1 1 617345A9
 P 5850 2100
@@
 $EndComp
 $Comp
-L power:GND #PWR0118
+L BoosterPack-rescue:GND-power #PWR0118
 U 1 1 61733D4A
 P 5850 1800
@@
 $EndComp
 $Comp
-L power:GND #PWR0119
+L BoosterPack-rescue:GND-power #PWR0119
 U 1 1 6173051A
 P 5850 1400
@@
 $EndComp
 $Comp
-L power:GND #PWR0120
+L BoosterPack-rescue:GND-power #PWR0120
 U 1 1 61748007
 P 1050 1450
@@
 $EndComp
 $Comp
-L power:GND #PWR0121
+L BoosterPack-rescue:GND-power #PWR0121
 U 1 1 61748F8F
 P 2250 1450
@@
 $EndComp
 $Comp
-L power:GND #PWR0122
+L BoosterPack-rescue:GND-power #PWR0122
 U 1 1 6174BD93
 P 1600 2950
@@
 	7250 2150 7550 2150
 $Comp
-L power:GND #PWR0123
+L BoosterPack-rescue:GND-power #PWR0123
 U 1 1 6175D652
 P 8650 1950
@@
 	7800 2950 7800 3450
 $Comp
-L Connector:TestPoint TP12
+L BoosterPack-rescue:TestPoint-Connector TP12
 U 1 1 617C0D53
 P 6600 3450
+AR Path="/617C0D53" Ref="TP12"  Part="1"
+AR Path="/61536750/617C0D53" Ref="TP12"  Part="1"
 F 0 "TP12" V 6795 3522 50  0000 C CNN
 F 1 "Keypad 1" V 6700 3600 50  0000 C CNN
@@
 $EndComp
 $Comp
-L Connector:TestPoint TP13
+L BoosterPack-rescue:TestPoint-Connector TP13
 U 1 1 617C1E13
 P 7200 3450
+AR Path="/617C1E13" Ref="TP13"  Part="1"
+AR Path="/61536750/617C1E13" Ref="TP13"  Part="1"
 F 0 "TP13" V 7395 3522 50  0000 C CNN
 F 1 "Keypad 2" V 7300 3600 50  0000 C CNN
@@
 $EndComp
 $Comp
-L Connector:TestPoint TP15
+L BoosterPack-rescue:TestPoint-Connector TP15
 U 1 1 617C4443
 P 7750 3450
+AR Path="/617C4443" Ref="TP15"  Part="1"
+AR Path="/61536750/617C4443" Ref="TP15"  Part="1"
 F 0 "TP15" V 7945 3522 50  0000 C CNN
 F 1 "Keypad 3" V 7850 3600 50  0000 C CNN
@@
 $EndComp
 $Comp
-L Connector:TestPoint TP16
+L BoosterPack-rescue:TestPoint-Connector TP16
 U 1 1 617C6A91
 P 8350 3450
+AR Path="/617C6A91" Ref="TP16"  Part="1"
+AR Path="/61536750/617C6A91" Ref="TP16"  Part="1"
 F 0 "TP16" V 8545 3522 50  0000 C CNN
 F 1 "Keypad 4" V 8450 3600 50  0000 C CNN
@@
 $EndComp
 $Comp
-L Connector:TestPoint TP17
+L BoosterPack-rescue:TestPoint-Connector TP17
 U 1 1 617C908C
 P 8850 3450
+AR Path="/617C908C" Ref="TP17"  Part="1"
+AR Path="/61536750/617C908C" Ref="TP17"  Part="1"
 F 0 "TP17" V 9045 3522 50  0000 C CNN
 F 1 "Keypad 5" V 8950 3600 50  0000 C CNN
@@
 $EndComp
 $Comp
-L Connector:TestPoint TP18
+L BoosterPack-rescue:TestPoint-Connector TP18
 U 1 1 617CB7E4
 P 9450 3450
+AR Path="/617CB7E4" Ref="TP18"  Part="1"
+AR Path="/61536750/617CB7E4" Ref="TP18"  Part="1"
 F 0 "TP18" V 9645 3522 50  0000 C CNN
 F 1 "Keypad 6" V 9550 3600 50  0000 C CNN
@@
 	9500 3450 9500 2950
 $Comp
-L Connector:TestPoint TP20
+L BoosterPack-rescue:TestPoint-Connector TP20
 U 1 1 617EBE74
 P 10050 3450
+AR Path="/617EBE74" Ref="TP20"  Part="1"
+AR Path="/61536750/617EBE74" Ref="TP20"  Part="1"
 F 0 "TP20" V 10245 3522 50  0000 C CNN
 F 1 "Keypad 7" V 10150 3600 50  0000 C CNN
@@
 $EndComp
 $Comp
-L Connector:TestPoint TP21
+L BoosterPack-rescue:TestPoint-Connector TP21
 U 1 1 617EEBE7
 P 10650 3450
+AR Path="/617EEBE7" Ref="TP21"  Part="1"
+AR Path="/61536750/617EEBE7" Ref="TP21"  Part="1"
 F 0 "TP21" V 10845 3522 50  0000 C CNN
 F 1 "Keypad 8" V 10750 3600 50  0000 C CNN
@@
 Control
 $Comp
-L Connector:TestPoint TP11
+L BoosterPack-rescue:TestPoint-Connector TP11
 U 1 1 6180A68B
 P 1650 4750
+AR Path="/6180A68B" Ref="TP11"  Part="1"
+AR Path="/61536750/6180A68B" Ref="TP11"  Part="1"
 F 0 "TP11" H 1708 4868 50  0000 L CNN
 F 1 "TestPoint - Electric Strike Control" H 1000 5000 50  0000 L CNN
@@
 	1950 1450 2150 1450
 $Comp
-L Connector:TestPoint TP7
+L BoosterPack-rescue:TestPoint-Connector TP7
 U 1 1 61828BFF
 P 1800 3100
+AR Path="/61828BFF" Ref="TP7"  Part="1"
+AR Path="/61536750/61828BFF" Ref="TP7"  Part="1"
 F 0 "TP7" H 1858 3218 50  0000 L CNN
 F 1 "TestPoint - GND Rechargeable Batteries" H 1000 3350 50  0000 L CNN
@@
 	1800 2950 2050 2950
 $Comp
-L Connector:TestPoint TP8
+L BoosterPack-rescue:TestPoint-Connector TP8
 U 1 1 6182F7F2
 P 2150 1350
+AR Path="/6182F7F2" Ref="TP8"  Part="1"
+AR Path="/61536750/6182F7F2" Ref="TP8"  Part="1"
 F 0 "TP8" H 2208 1468 50  0000 L CNN
 F 1 "TestPoint - GND VCC" H 1750 1600 50  0000 L CNN
@@
 	2150 1450 2250 1450
 $Comp
-L Connector:TestPoint TP14
+L BoosterPack-rescue:TestPoint-Connector TP14
 U 1 1 61839E0C
 P 7550 1900
+AR Path="/61839E0C" Ref="TP14"  Part="1"
+AR Path="/61536750/61839E0C" Ref="TP14"  Part="1"
 F 0 "TP14" H 7608 2018 50  0000 L CNN
 F 1 "GND Keypad" H 7608 1927 50  0000 L CNN
@@
 	7550 2150 7800 2150
 $Comp
-L Connector:TestPoint TP19
+L BoosterPack-rescue:TestPoint-Connector TP19
 U 1 1 61841CC3
 P 9750 1900
+AR Path="/61841CC3" Ref="TP19"  Part="1"
+AR Path="/61536750/61841CC3" Ref="TP19"  Part="1"
 F 0 "TP19" H 9808 2018 50  0000 L CNN
 F 1 "GND Keypad" H 9808 1927 50  0000 L CNN
